File: boards/ADNS-9800.brd (EAGLE design)
At the start: 32.7 x 32.5 mm, 27 parts, among them Q1 TRANSISTOR_SC-75

Commit message: put all the downloaded files into directories
Parts:
- removed R1, R2, R4: 1.8K, SparkFun-Passives:0603-RES
- removed R3, R5, R6: 3.3K, SparkFun-Passives:0603-RES
- removed SJ1, SJ3, SJ6: SOLDERJUMPERTRACE, SparkFun-Passives:SJ_2S-TRACE
- removed SJ2, SJ4, SJ5: SOLDERJUMPERNO, SparkFun-Passives:SJ_2S-NO
- moved JP1 0.28 mm to (15.7, 27.5)
Connections:
- removed net MOSI-H: JP1.5, R1.1, SJ1.1
- removed net N$11: R3.1, SJ2.2
- removed net N$15: R5.1, SJ5.2
- removed net N$9: R6.1, SJ4.2
- removed net SCK: R2.2, SJ2.1, SJ3.2, U$1.P$5
- removed net SCK-H: JP1.3, R2.1, SJ3.1
- removed net SS-H: JP1.7, R4.1, SJ6.1
- new net SCLK: JP1.5, U$1.P$5
- net AGND: now also JP1.3; no longer JP1.4, R3.2, R5.2, R6.2
- net DGND: now also JP1.2; no longer JP1.6
- net MISO: now also JP1.8; no longer JP1.1
- net MOSI: now also JP1.7; no longer R1.2, SJ1.2, SJ4.1
- net MOTION: now also JP1.4; no longer JP1.8
- net SS: now also JP1.6; no longer R4.2, SJ5.1, SJ6.2
- net VIN: now also JP1.1; no longer JP1.2
Routing:
- net SS: track 59.2 -> 5.56 mm
- net SCK: track 41.1 -> 0.00 mm
- net MOSI-H: track 39.9 -> 0.00 mm
- net SCK-H: track 33.6 -> 0.00 mm
- net MOSI: track 35.1 -> 7.38 mm, vias 1 -> 0
- net SS-H: track 25.4 -> 0.00 mm, vias 1 -> 0
- net DGND: track 18.3 -> 9.15 mm, vias 3 -> 0
- net N$2: track 16.3 -> 24.5 mm, vias 0 -> 1
- net SCLK: track 0.00 -> 7.70 mm
- net MOTION: track 4.35 -> 11.7 mm
- net N$15: track 5.94 -> 0.00 mm, vias 1 -> 0
- net N$11: track 4.60 -> 0.00 mm, vias 1 -> 0
- net N$9: track 3.70 -> 0.00 mm, vias 1 -> 0
- net AGND: track 4.01 -> 1.30 mm, vias 2 -> 0
- net LSR_NEN: track 10.9 -> 13.1 mm
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Other:
- board text removed: "06/2013"
- board text removed: "3.3V"
- board text removed: "5V"
- board text removed: "MrJohnK"
- board text removed: "v2.0"
