File: boards/OpenPad.brd (EAGLE design)
At the start: 53.3 x 42 mm, 54 parts, among them P1 P1, P2 P2, P3 P3, P4 P4, Q1 16MHz, U1 4066D, U2 ATMEGA32U4TQFP

Commit message: put all the downloaded files into directories
Parts:
- added C1: 1uF, SparkFun-Capacitors:0402-CAP
- added TP1: AREF, SparkFun-Passives:PAD.02X.02
Connections:
- new net N$24: TP1.P$1, U2.42
- new net N$25: C1.2, U2.6
- net GND: now also C1.1
Changed lines of the file:
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@@
 <element name="SJ20" library="jumper" package="SJW" value="" x="48.26" y="8.89" rot="R90"/>
 <element name="SJ16" library="jumper" package="SJW" value="" x="33.02" y="33.02" rot="R270"/>
+<element name="TP1" library="SparkFun-Passives" package="PAD.02X.02" value="AREF" x="0" y="-15.24"/>
+<element name="C1" library="SparkFun-Capacitors" package="0402-CAP" value="1uF" x="1.27" y="-17.78">
+<attribute name="PROD_ID" value="CAP-00810" x="1.27" y="-17.78" size="1.778" layer="27" display="off"/>
+</element>
 </elements>
 <signals>
@@
 <contactref element="Q1" pad="2"/>
 <contactref element="SJ20" pad="2"/>
-<wire x1="2.54" y1="-11.43" x2="48.26" y2="10.16" width="0" layer="19" extent="1-1"/>
-<wire x1="6.35" y1="-3.81" x2="2.54" y2="-11.43" width="0" layer="19" extent="1-1"/>
-<wire x1="3.81" y1="8.89" x2="6.35" y2="-3.81" width="0" layer="19" extent="16-16"/>
-<wire x1="15.24" y1="20.3708" x2="6.97" y2="12.7" width="0" layer="19" extent="1-16"/>
-<wire x1="21.59" y1="13.97" x2="15.24" y2="20.3708" width="0" layer="19" extent="16-16"/>
-<wire x1="24.13003125" y1="14.61998125" x2="21.59" y2="13.97" width="0" layer="19" extent="16-16"/>
-<wire x1="27.9260375" y1="18.348475" x2="24.13" y2="15.24" width="0" layer="19" extent="1-16"/>
-<wire x1="38.1" y1="19.67" x2="34.29" y2="20.955" width="0" layer="19" extent="1-16"/>
-<wire x1="39.37" y1="19.67" x2="38.1" y2="19.67" width="0" layer="19" extent="16-16"/>
+<contactref element="C1" pad="1"/>
+<wire x1="39.37" y1="23.51" x2="38.1" y2="23.51" width="0" layer="19" extent="16-16"/>
+<wire x1="39.37" y1="19.67" x2="39.37" y2="23.51" width="0" layer="19" extent="16-16"/>
+<wire x1="38.1" y1="19.67" x2="39.37" y2="19.67" width="0" layer="19" extent="16-16"/>
 <wire x1="41.21964375" y1="17.782790625" x2="39.37" y2="19.67" width="0" layer="19" extent="1-16"/>
-<wire x1="38.1" y1="23.51" x2="38.1" y2="19.67" width="0" layer="19" extent="16-16"/>
-<wire x1="39.37" y1="23.51" x2="38.1" y2="23.51" width="0" layer="19" extent="16-16"/>
+<wire x1="34.29" y1="20.955" x2="38.1" y2="19.67" width="0" layer="19" extent="1-16"/>
+<wire x1="24.13" y1="15.24" x2="27.9260375" y2="18.348475" width="0" layer="19" extent="1-16"/>
+<wire x1="21.59" y1="13.97" x2="24.13003125" y2="14.61998125" width="0" layer="19" extent="16-16"/>
+<wire x1="15.24" y1="20.3708" x2="21.59" y2="13.97" width="0" layer="19" extent="16-16"/>
+<wire x1="48.26" y1="10.16" x2="41.21964375" y2="17.782790625" width="0" layer="19" extent="1-1"/>
+<wire x1="6.97" y1="12.7" x2="15.24" y2="20.3708" width="0" layer="19" extent="1-16"/>
+<wire x1="6.35" y1="-3.81" x2="3.81" y2="8.89" width="0" layer="19" extent="16-16"/>
+<wire x1="2.54" y1="-11.43" x2="6.35" y2="-3.81" width="0" layer="19" extent="1-1"/>
+<wire x1="0.62" y1="-17.78" x2="2.54" y2="-11.43" width="0" layer="19" extent="1-1"/>
 </signal>
 <signal name="VCC">
@@
 <wire x1="31.885834375" y1="22.308275" x2="22.86" y2="31.75" width="0" layer="19" extent="1-1"/>
 </signal>
+<signal name="N$24">
+<contactref element="U2" pad="42"/>
+<contactref element="TP1" pad="P$1"/>
+<wire x1="0" y1="-15.24" x2="28.491721875" y2="18.9141625" width="0" layer="19" extent="1-1"/>
+</signal>
+<signal name="N$25">
+<contactref element="U2" pad="6"/>
+<contactref element="C1" pad="2"/>
+<wire x1="1.92" y1="-17.78" x2="30.188778125" y2="12.408778125" width="0" layer="19" extent="1-1"/>
+</signal>
 </signals>
