File: boards/aixplorer_battery_pack.brd (EAGLE design)
At the start: 40 x 11 mm, 7 parts

Commit message: put all the downloaded files into directories
Parts:
- removed TP1, TP2, TP3, TP4, TP5: TPTP15R, testpad:TP15R
- turned U$1 to 180 degrees
Connections:
- new net ACC: U$1.P$21, U$2.P$1
- new net AUDIO: U$1.P$11, U$2.P$11
- net 3V3: now also U$2.P$10; no longer TP1.TP
- net 5V: no longer U$2.P$6
- net D+: now also U$2.P$6; no longer U$2.P$1, U$2.P$5
- net D-: now also U$2.P$5; no longer U$2.P$3, U$2.P$7
- net GND: now also U$2.P$9; no longer U$2.P$4, U$2.P$8
- net LOUT: now also U$2.P$7; no longer TP4.TP
- net ROUT: now also U$2.P$8; no longer TP5.TP
- net RX: now also U$2.P$4; no longer TP2.TP
- net TX: now also U$2.P$3; no longer TP3.TP
Routing:
- net ACC: track 0.00 -> 20.8 mm
- net AUDIO: track 0.00 -> 19.8 mm, vias 0 -> 1
- net D+: track 27.7 -> 14.8 mm, vias 1 -> 0
- net 5V: track 23.5 -> 16.8 mm, vias 1 -> 0
- net D-: track 14.4 -> 18.8 mm, vias 1 -> 0
- net N$2: track 0.00 -> 4.00 mm
- net N$1: track 0.00 -> 4.00 mm
- net RX: track 19.3 -> 23.1 mm
- net ROUT: track 14.6 -> 17.4 mm
- net LOUT: track 12.0 -> 14.6 mm
- net GND: track 33.6 -> 31.2 mm, vias 1 -> 0
- net 3V3: track 18.8 -> 16.9 mm
- net TX: track 19.3 -> 19.2 mm, vias 0 -> 1
Other:
- outline, holes or cut-outs redrawn
- board text added: "TOP"
