File: boards/control_board.brd (EAGLE design)
At the start: 63.5 x 19.1 mm, 16 parts

Commit message: put all the downloaded files into directories
Parts:
- removed JP1: (no value), SparkFun-Connectors:JST-2-SMD
- removed JP2, JP5: (no value), SparkFun-Connectors:1X06_LOCK
- removed STANDOFF2, STANDOFF3: STAND-OFF, SparkFun-Electromechanical:STAND-OFF
- removed TLC5947: TLC5947DAP, SparkFun-DigitalIC:DAP
- removed U$2, U$3, U$4, U$5, U$6, U$7, U$8: SWR204-D02, SparkFun-Connectors:SWR204
- added ANT1: PIFA-2.4GHZ, berkeley-epic:PIFA-2.4GHZ
- added BLE1: HM10_BLE, pecs:HM10
- added C10, C11, C12, C13, C4, C5, C6, C7, C8: 100nF, pecs:0805
- added C2, C3: 1uF, pecs:0805
- added C9: 10uF, pecs:0805
- added D1, D2, D3, D4, D5: (no value), berkeley-epic:LED-1206
- added IC1: FT232RL, ftdichip:SSOP28
- added J1, J9: HD.1-6, pecs:HD.1-6
- added J10: ICSP_HDR, pecs:H.1-6
- added J11: HD.1-14, pecs:HD.1-16
- added J12, J7: JTAG, pecs:JTAG
- added J13: HD.1-12, pecs:HD.1-12
- added J2, J3, J4, J5, J6: (no value), pecs:H.1-2
- added J8: EPIC-PROG-PORT, berkeley-epic:HEADER2X3X2MM
- added Q1, Q2, Q3, Q4, Q5: NFET_DPAK, pecs:DPAK
- added R10, R5, R6, R7, R8, R9: (no value), pecs:1206
- added R11, R12, R13, R22, R3: 10k, pecs:0805
- added R14: 1k8, pecs:0805
- added R15, R16, R17, R18, R20, R21, R24: 4k7, pecs:0805
- added R2: 2k, pecs:0805
- added R23, R4: 100k, pecs:0805
- added U1: PIC24FJ32GB004, pecs:TQFP44
- added U2: OKI-78SR_3V3_SMPS, pecs:SMPS_MODULE
- added U3: NUMONYX_FLASH, pecs:NUMONYX_FLASH
- added U4: EPIC-CORE_A, berkeley-epic:EPIC-LCC68
- C1: value .1uF -> 10uF; device SparkFun-Capacitors:0603-CAP -> pecs:0805
- R1: value 1.8k -> 10k; device SparkFun-Resistors:0603-RES -> pecs:0805
- U$1: value SWR204-D02 -> USB_B; device SparkFun-Connectors:SWR204 -> pecs:USB_MOLEX_7041
- moved C1 126.6 mm to (-76.7, 63.6), turned to 180 degrees
- moved R1 120.6 mm to (-77.9, 47.4)
- moved U$1 44.3 mm to (-35.1, 8.19), turned to 0 degrees
Connections:
- removed net BLANK: JP2.4, JP5.4, TLC5947.2
- removed net OUT0: TLC5947.5, U$1.P$3
- removed net OUT1: TLC5947.6, U$1.P$2
- removed net OUT10: TLC5947.15, U$4.P$2
- removed net OUT11: TLC5947.16, U$4.P$1
- removed net OUT12: TLC5947.17, U$5.P$3
- removed net OUT13: TLC5947.18, U$5.P$2
- removed net OUT14: TLC5947.19, U$5.P$1
- removed net OUT15: TLC5947.20, U$6.P$3
- removed net OUT16: TLC5947.21, U$6.P$2
- removed net OUT17: TLC5947.22, U$6.P$1
- removed net OUT18: TLC5947.23, U$7.P$3
- removed net OUT19: TLC5947.24, U$7.P$2
- removed net OUT2: TLC5947.7, U$1.P$1
- removed net OUT20: TLC5947.25, U$7.P$1
- removed net OUT21: TLC5947.26, U$8.P$3
- removed net OUT22: TLC5947.27, U$8.P$2
- removed net OUT23: TLC5947.28, U$8.P$1
- removed net OUT3: TLC5947.8, U$3.P$3
- removed net OUT4: TLC5947.9, U$3.P$2
- removed net OUT5: TLC5947.10, U$3.P$1
- removed net OUT6: TLC5947.11, U$2.P$3
- removed net OUT7: TLC5947.12, U$2.P$2
- removed net OUT8: TLC5947.13, U$2.P$1
- removed net OUT9: TLC5947.14, U$4.P$3
- removed net SCLK: JP2.5, JP5.5, TLC5947.3
- removed net SIN: JP2.6, TLC5947.4
- removed net SOUT: JP5.6, TLC5947.29
- removed net VCC: C1.1, JP2.1, JP5.1, TLC5947.32
- removed net VDD: JP1.2, U$1.P$4, U$2.P$4, U$3.P$4, U$4.P$4, U$5.P$4, U$6.P$4, U$7.P$4, U$8.P$4
- removed net XLAT: JP2.3, JP5.3, TLC5947.30
- new net +14V: C1.2, J1.P1, J2.P1, J3.P1, J6.P1, R1.2, U2.VIN
- new net +3V3: BLE1.P$12, C11.2, C12.2, C13.2, C2.2, C3.2, C4.2, C5.2, C6.2, C7.2, D1.A, D2.A, D3.A, D4.A, D5.A, IC1.20, IC1.4, J1.P2, J10.P2, J11.P1, J11.P14, J12.VDD, J13.P1, J4.P1, J5.P1, J7.VDD, J8.1, J9.P1, R15.1, R23.1, R4.1, U1.10, U1.17, U1.28, U1.40, U1.42, U2.VOUT, U3.1, U3.13/7, U3.14/8, U3.2, U3.5/3, U3.9, U4.P$17, U4.P$34, U4.P$37, U4.P$51, U4.P$68
- new net +5V: R24.2, U$1.1_VBUS
- new net ACTL0: J11.P3, U4.P$21
- new net ACTL1: J11.P4, U4.P$22
- new net ACTL2: J11.P5, U4.P$23
- new net ACTL3: J11.P6, U4.P$24
- new net ACTL4: J11.P7, U4.P$25
- new net ACTL5: J11.P8, U4.P$26
- new net AUX_RX: J1.P6, U1.22
- new net AUX_TX: J1.P4, U1.21
- new net BLEGPIO: BLE1.P$27, U4.P$5
- new net BLE_CTS: BLE1.P$3, U1.32
- new net BLE_RTS: BLE1.P$4, U1.31
- new net BLE_RX: BLE1.P$2, U1.11
- new net BLE_TX: BLE1.P$1, U1.5
- new net BL_CTL: J13.P10, U1.3
- new net CB0: IC1.23, R20.1
- new net CB1: IC1.22, R21.1
- new net CMCLR: C10.2, J10.P1, R23.2, U1.18
- new net C_INT0: U1.43, U4.P$20
- new net DCTL0: J11.P9, U4.P$30
- new net DCTL1: J11.P10, U4.P$31
- new net DCTL2: J11.P11, U4.P$32
- new net DCTL3: J11.P12, U4.P$33
- new net E_U1RX: J8.4, U1.15, U4.P$62
- new net E_U1TX: J8.3, U1.14, U4.P$61
- new net FAN_NEG: J2.P2, Q1.TAG, R10.2, R5.2, R6.2, R7.2, R8.2, R9.2
- new net FC_A: Q1.P1, R11.2, U4.P$6
- new net FC_B: Q2.P1, R12.2, U4.P$7
- new net FC_C: Q3.P1, R13.2, U4.P$8
- new net FL_CLK: J12.TCK, U1.36, U3.12/6, U3.16
- new net FL_CS: J12.TMS, U1.30, U3.3/1, U3.7
- new net FL_MISO: J12.TDO, U1.38, U3.4/2, U3.8
- new net FL_MOSI: J12.TDI, U1.37, U3.11/5, U3.15
- new net FT_CTS: IC1.11, U1.13
- new net FT_RX: IC1.5, U1.20
- new net FT_TX: IC1.1, U1.19
- new net HC: Q4.P1, R14.2, U1.2
- new net HEAT_NEG: J6.P2, Q4.TAG
- new net LCD_EN: Q5.P1, R3.2, U1.41
- new net LCD_GND: J13.P11, Q5.TAG
- new net LCD_RST: J13.P9, U1.35
- new net L_SPI_CLK: J13.P3, U1.25
- new net L_SPI_LCD_CS: J13.P7, U1.23
- new net L_SPI_MISO: J13.P5, U1.27
- new net L_SPI_MOSI: J13.P4, U1.26
- new net L_SPI_TP_CS: J13.P6, U1.24
- new net N$10: D1.C, R16.2
- new net N$11: D2.C, R17.2
- new net N$12: D3.C, R18.2
- new net N$13: R16.1, U4.P$65
- new net N$14: D5.C, R21.2
- new net N$15: R17.1, U4.P$66
- new net N$16: R18.1, U4.P$67
- new net N$19: IC1.19, R22.2, R24.1
- new net N$23: R1.1, R2.2, U4.P$19
- new net N$3: ANT1.P$1, U4.P$43
- new net N$6: Q2.TAG, R5.1, R6.1, R9.1
- new net N$7: Q3.TAG, R10.1, R7.1, R8.1
- new net N$9: D4.C, R20.2
- new net PGC: J10.P5, U1.9
- new net PGD: J10.P4, U1.8
- new net RESETB: BLE1.P$11, R15.2, U1.34
- new net RH_CLK: J9.P5, U1.44
- new net RH_DAT: J9.P6, U1.1
- new net RST: C8.2, J8.6, R4.2, U4.P$16
- new net SYSKEY: BLE1.P$23, U1.12
- new net TCK: J7.TCK, J8.5, U4.P$15
- new net TDI: J7.TDI, U4.P$13
- new net TDO: J7.TDO, U4.P$12
- new net TMS: J7.TMS, U4.P$14
- new net TP_IRQ: J13.P8, U1.33, U4.P$38
- new net USBD_N: IC1.16, U$1.2_D-
- new net USBD_P: IC1.15, U$1.3_D+
- net GND: now also ANT1.P$2, ANT1.P$3, BLE1.P$13, BLE1.P$14, BLE1.P$21, BLE1.P$22, C1.1, C10.1, C11.1, C12.1, C13.1, C2.1, C3.1, C4.1, C5.1, C6.1, C7.1, C8.1, C9.1, IC1.18, IC1.21, IC1.25, IC1.26, IC1.7, J1.P5, J10.P3, J11.P13, J11.P2, J12.GND, J13.P12, J13.P2, J3.P2, J4.P2, J5.P2, J7.GND, J8.2, J9.P2, Q1.P3, Q2.P3, Q3.P3, Q4.P3, Q5.P3, R11.1, R12.1, R13.1, R14.1, R2.1, R22.1, R3.1, U$1.4_GND, U1.16, U1.29, U1.39, U1.6, U2.GND, U3.10, U3.6/4, U4.P$1, U4.P$18, U4.P$35, U4.P$42, U4.P$44, U4.P$52; no longer C1.2, JP1.1, JP2.2, JP5.2, R1.1, TLC5947.1, TLC5947.GND
- net N$1: now also C9.2, U1.7; no longer R1.2, TLC5947.31
Routing:
- net GND: track 10.9 -> 225.0 mm, vias 2 -> 54
- net BLE_RX: track 0.00 -> 130.4 mm, vias 0 -> 2
- net +3V3: track 0.00 -> 116.6 mm, vias 0 -> 19
- net +14V: track 0.00 -> 111.4 mm
- net TP_IRQ: track 0.00 -> 103.1 mm, vias 0 -> 4
- net SCLK: track 88.3 -> 0.00 mm
- net BLANK: track 88.1 -> 0.00 mm
- net E_U1RX: track 0.00 -> 87.9 mm, vias 0 -> 2
- net XLAT: track 87.6 -> 0.00 mm
- net BLE_TX: track 0.00 -> 78.8 mm, vias 0 -> 4
- net E_U1TX: track 0.00 -> 77.7 mm, vias 0 -> 3
- net VDD: track 71.7 -> 0.00 mm, vias 1 -> 0
- net BLEGPIO: track 0.00 -> 71.7 mm
- net FL_MOSI: track 0.00 -> 66.7 mm, vias 0 -> 2
- net BLE_CTS: track 0.00 -> 62.0 mm, vias 0 -> 2
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- added copper zone on layer 15, net +3V3
- added copper zone on layer 1, net GND
- added copper zone on layer 2, net GND
Other:
- board size 63.5 x 19.1 mm -> 60 x 114 mm
- board text added: "+"
- board text added: "EPIC"
- board text added: "FAN"
- board text added: "FLASH"
- board text added: "HEAT"
- board text added: "ICSP"
- board text added: "M ANDERSEN (C) 2013"
- board text added: "PECS CTL 2.0"
- board text added: "UC BERKELEY"
- board text removed: "0, 1, 2"
- board text removed: "12, 13, 14"
- board text removed: "15, 16, 17"
- board text removed: "18, 19, 20"
- board text removed: "21, 22, 23"
- board text removed: "3, 4, 5"
- board text removed: "6, 7, 8"
- board text removed: "9, 10, 11"
- board text removed: "GND VDD"
- board text removed: "v1.2"
- board text removed: "vcc gnd xlat blank sclk sin"
- board text removed: "vcc gnd xlat blank sclk sout"
