File: boards/femto.brd (EAGLE design)
At the start: 50.2 x 25.1 mm, 29 parts, among them IC1 MEGA8-AI, J1 RJ12RIGHTANGLE-I2C, J2 RJ12RIGHTANGLE-I2C

Commit message: put all the downloaded files into directories
Routing:
- net RESET: track 0.00 -> 4.94 mm
- net SCK: track 4.15 -> 0.00 mm
- net GND: track 101.2 -> 102.2 mm
