File: boards/fnordstripe.brd (EAGLE design)
At the start: 31.8 x 31.8 mm, 23 parts, among them IC2 78L05Z, IC3 MEGA8-AI, Q1 16MHz, Q2 IRF540, Q3 IRF540, Q4 IRF540

Commit message: put all the downloaded files into directories
Parts:
- turned ISP to 0 degrees
Connections:
- net +5V: now also ISP.5; no longer ISP.2
- net GND: now also ISP.1; no longer ISP.6
- net MISO: now also ISP.6; no longer ISP.1
- net MOSI: now also ISP.3; no longer ISP.4
- net RST: now also ISP.2; no longer ISP.5
- net SCK: now also ISP.4; no longer ISP.3
Changed lines of the file:
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@@
 <attribute name="NAME" x="20.2946" y="18.7706" size="1.27" layer="25" ratio="12" rot="R180"/>
 </element>
-<element name="ISP" library="con-lstb" package="MA03-2" value="" x="27.432" y="28.702" smashed="yes" rot="R180">
-<attribute name="OC_NEWARK" value="unknown" x="27.432" y="28.702" size="1.778" layer="27" rot="R180" display="off"/>
-<attribute name="MPN" value="" x="27.432" y="28.702" size="1.778" layer="27" rot="R180" display="off"/>
-<attribute name="MF" value="" x="27.432" y="28.702" size="1.778" layer="27" rot="R180" display="off"/>
-<attribute name="OC_FARNELL" value="unknown" x="27.432" y="28.702" size="1.778" layer="27" rot="R180" display="off"/>
-<attribute name="NAME" x="31.496" y="34.544" size="1.27" layer="25" ratio="10" rot="R180"/>
-<attribute name="VALUE" x="28.702" y="32.893" size="1.27" layer="27" ratio="10" rot="R180"/>
+<element name="ISP" library="con-lstb" package="MA03-2" value="" x="27.432" y="28.702" smashed="yes">
+<attribute name="OC_NEWARK" value="unknown" x="27.432" y="28.702" size="1.778" layer="27" display="off"/>
+<attribute name="MPN" value="" x="27.432" y="28.702" size="1.778" layer="27" display="off"/>
+<attribute name="MF" value="" x="27.432" y="28.702" size="1.778" layer="27" display="off"/>
+<attribute name="OC_FARNELL" value="unknown" x="27.432" y="28.702" size="1.778" layer="27" display="off"/>
+<attribute name="NAME" x="23.368" y="22.86" size="1.27" layer="25" ratio="10"/>
+<attribute name="VALUE" x="26.162" y="24.511" size="1.27" layer="27" ratio="10"/>
 </element>
 <element name="SV3" library="con-lstb" package="MA04-1" value="" x="4.445" y="19.177" smashed="yes" rot="R270">
@@
 <contactref element="Q3" pad="S"/>
 <wire x1="22.196825" y1="10.385825" x2="24.228825" y2="10.385825" width="0.4064" layer="1"/>
-<contactref element="ISP" pad="6"/>
+<contactref element="ISP" pad="1"/>
 <wire x1="25.381" y1="21.9456" x2="25.381" y2="22.841" width="0.4064" layer="1"/>
 <wire x1="25.381" y1="22.841" x2="25.527" y2="22.987" width="0.4064" layer="1"/>
@@
 <wire x1="23.781" y1="13.3604" x2="23.781" y2="14.764" width="0.4064" layer="1"/>
 <wire x1="23.781" y1="14.764" x2="24.162" y2="15.145" width="0.4064" layer="1"/>
-<contactref element="ISP" pad="2"/>
+<contactref element="ISP" pad="5"/>
 <wire x1="29.972" y1="25.527" x2="29.972" y2="27.432" width="0.4064" layer="1"/>
 <wire x1="24.581" y1="21.9456" x2="24.581" y2="25.597" width="0.4064" layer="1"/>
@@
 <wire x1="21.4884" y1="14.853" x2="21.717" y2="14.6244" width="0.3048" layer="1"/>
 <wire x1="21.717" y1="14.6244" x2="21.717" y2="13.589" width="0.3048" layer="1"/>
-<contactref element="ISP" pad="1"/>
+<contactref element="ISP" pad="6"/>
 <wire x1="26.289" y1="24.638" x2="28.702" y2="27.051" width="0.3048" layer="16"/>
 <wire x1="28.702" y1="27.051" x2="28.702" y2="28.702" width="0.3048" layer="16"/>
@@
 <contactref element="IC3" pad="17"/>
 <wire x1="22.9556" y1="13.335" x2="22.981" y2="13.3604" width="0.3048" layer="1"/>
-<contactref element="ISP" pad="3"/>
+<contactref element="ISP" pad="4"/>
 <wire x1="27.432" y1="29.972" x2="26.162" y2="28.702" width="0.3048" layer="16"/>
 <wire x1="26.162" y1="28.702" x2="26.162" y2="27.051" width="0.3048" layer="16"/>
@@
 <wire x1="24.003" y1="18.034" x2="30.0546" y2="18.034" width="0.3048" layer="1"/>
 <wire x1="30.0546" y1="18.034" x2="30.0736" y2="18.053" width="0.3048" layer="1"/>
-<contactref element="ISP" pad="5"/>
+<contactref element="ISP" pad="2"/>
 <wire x1="21.971" y1="29.972" x2="24.892" y2="29.972" width="0.4064" layer="16"/>
 <wire x1="23.495" y1="28.448" x2="21.971" y2="29.972" width="0.3048" layer="16"/>
@@
 <signal name="MOSI">
 <contactref element="IC3" pad="15"/>
-<contactref element="ISP" pad="4"/>
+<contactref element="ISP" pad="3"/>
 <wire x1="27.432" y1="27.432" x2="25.654" y2="25.654" width="0.3048" layer="16"/>
 <wire x1="25.654" y1="25.654" x2="25.654" y2="16.764" width="0.3048" layer="16"/>
