File: boards/tinyRF.brd (EAGLE design)
At the start: 18 x 13 mm, 23 parts

Commit message: put all the downloaded files into directories
Parts:
- removed U$1: CYRF69103, JCM:QFN40
- removed _SS: SOLDER_PAD.05X.05, JCM:SOLDER_PAD_.05X.05
- added !SS: SOLDER_PADTH, JCM-Connectors:1X1_50MIL
- added CYRF6936: CYRF6936QFN, JCM-IC:QFN50P600X600X90-41N
- C1, C10, C11, C15, C3, C4, C5, C6, C7, C8, C9: device SparkFun-Passives:0402-CAP -> JCM-Capacitors:0402-CAP
- C14: device SparkFun-Passives:0805 -> JCM-Capacitors:0805
- GND, IRQ, MISO, MOSI, SCK, VCC: value SOLDER_PAD.05X.05 -> SOLDER_PADTH; device JCM:SOLDER_PAD_.05X.05 -> JCM-Connectors:1X1_50MIL
- moved VCC 3.16 mm to (12.7, 19.7)
- moved C15 2.29 mm to (16.0, 16.3)
- moved MISO 1.91 mm to (12.7, 21.0)
- moved C14 1.86 mm to (13.2, 17.4)
- moved MOSI 1.53 mm to (12.7, 22.2)
- moved C8 1.51 mm to (13.4, 16.3)
- moved IRQ 1.15 mm to (12.7, 23.5)
- moved C9 0.89 mm to (21.0, 16.3)
- moved SCK 0.77 mm to (12.7, 24.8)
- moved C5 0.69 mm to (18.5, 16.3)
- moved C11 0.30 mm to (22.9, 22.6)
- moved C7 0.29 mm to (22.9, 17.6)
- moved C1 0.23 mm to (21.8, 26.8)
- moved C10 0.20 mm to (22.9, 20.1)
- moved GND 0.13 mm to (12.7, 27.3)
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Connections:
- removed net N$4: U$1.21
- removed net N$5: U$1.22
- new net PACTL: CYRF6936.30
- new net TV1: CYRF6936.29
- net GND: now also CYRF6936.12, CYRF6936.14, CYRF6936.15, CYRF6936.17, CYRF6936.18, CYRF6936.19, CYRF6936.2, CYRF6936.20, CYRF6936.21, CYRF6936.22, CYRF6936.23, CYRF6936.31, CYRF6936.32, CYRF6936.36, CYRF6936.37, CYRF6936.39, CYRF6936.4, CYRF6936.41, CYRF6936.5, CYRF6936.9, GND.1; no longer GND.P$1, U$1.12, U$1.14, U$1.17, U$1.18, U$1.20, U$1.37, U$1.GND
- net IRQ: now also CYRF6936.26, IRQ.1; no longer IRQ.P$1, U$1.27
- net MISO: now also CYRF6936.28, MISO.1; no longer MISO.P$1, U$1.29
- net MOSI: now also CYRF6936.27, MOSI.1; no longer MOSI.P$1, U$1.28
- net N$2: now also CYRF6936.1; no longer U$1.2
- net RFBIAS: now also CYRF6936.10; no longer U$1.10
- net RFN: now also CYRF6936.13; no longer U$1.13
- net RFP: now also CYRF6936.11; no longer U$1.11
- net RST: now also CYRF6936.34; no longer U$1.34
- net SCK: now also CYRF6936.25, SCK.1; no longer SCK.P$1, U$1.26
- net VCC: now also CYRF6936.16, CYRF6936.3, CYRF6936.33, CYRF6936.38, CYRF6936.40, CYRF6936.6, CYRF6936.7, CYRF6936.8, VCC.1; no longer U$1.16, U$1.3, U$1.33, U$1.39, U$1.40, U$1.6, U$1.7, U$1.9, VCC.P$1
- net VDD: now also CYRF6936.35; no longer U$1.36
- net _SS: now also !SS.1, CYRF6936.24; no longer U$1.25, _SS.P$1
Routing:
- net GND: track 3.92 -> 34.3 mm, vias 28 -> 46
- net VCC: track 42.4 -> 50.8 mm
- net SCK: track 2.84 -> 4.43 mm
- net RFN: track 1.01 -> 2.58 mm
- net IRQ: track 2.59 -> 3.67 mm
- net RST: track 3.49 -> 2.55 mm
- net RFP: track 3.48 -> 4.19 mm
- net _SS: track 4.42 -> 5.12 mm
- net MOSI: track 2.41 -> 2.94 mm
- net MISO: track 2.08 -> 2.58 mm
Other:
- board size 18 x 13 mm -> 13 x 13 mm
