File: boards/usbB_isp_no_lm2940.brd (EAGLE design)
At the start: 100 x 80 mm, 9 parts, among them IC2 TINY13-20PU, X1 PN61729-S

Commit message: put all the downloaded files into directories
Parts:
- moved R4 4.47 mm to (26.2, 14.6)
- moved X1 4.41 mm to (2.47, 8.94)
- moved R1 4.35 mm to (38.7, 13.5)
- moved C3 4.35 mm to (44.4, 5.65)
- moved IC2 4.35 mm to (37.2, 6.20)
- moved LED1 4.35 mm to (14.6, 9.03)
- moved R2 4.35 mm to (26.2, 12.0)
- moved SV2 4.35 mm to (49.3, 9.03)
- moved R3 4.35 mm to (26.5, 5.84)
Connections:
- net GND: now also X1.4
Routing:
- net VCC: track 79.7 -> 69.3 mm
Other:
- board size 100 x 80 mm -> 56 x 20 mm
